File: Medidor_Digital_Doble_Add1.kicad_pcb (KiCad board)
At the start: 2 copper layers, 0 parts

Commit message: Se termina el PCB, pero se requiere una PCB de menor tamaño y a una cara.
Parts:
- added C1: 100n, 1-Capacitor:C_0805_2012Metric, F.Cu at (129.1, 105.0)
- added C2: 100n, 1-Capacitor:C_0805_2012Metric, F.Cu at (135.5, 102.1)
- added J1: Screw_Terminal_01x01, 1-Pad:PAD_2.54_1.0, F.Cu at (136.8, 115.9)
- added J2: Screw_Terminal_01x01, 1-Pad:PAD_2.54_1.0, F.Cu at (130.9, 115.9)
- added J3: Screw_Terminal_01x01, 1-Pad:PAD_2.54_1.0, F.Cu at (121.4, 102.1)
- added J4: Screw_Terminal_01x01, 1-Pad:PAD_2.54_1.0, F.Cu at (121.4, 111.0)
- added J5: Screw_Terminal_01x01, 1-Pad:PAD_2.54_1.0, F.Cu at (121.4, 115.4)
- added J6: Screw_Terminal_01x01, 1-Pad:PAD_2.54_1.0, F.Cu at (121.4, 106.5)
- added R3: 1k2, 1-Resistor:R_0805_2012Metric, F.Cu at (136.4, 113.0)
- added R4: 1k2, 1-Resistor:R_0805_2012Metric, F.Cu at (131.7, 113.0)
- added R5: 330k, 1-Resistor:R_0805_2012Metric, F.Cu at (134.1, 109.9)
- added U1: INA823, 1-Package_SO:SOIC-8_3.9x4.9mm_P1.27mm, F.Cu at (134.0, 106.0)
Routing:
- net V1: track 0.00 -> 25.6 mm, vias 0 -> 1
- net -5V: track 0.00 -> 22.6 mm
- net AC2: track 0.00 -> 17.7 mm
- net AC1: track 0.00 -> 14.3 mm
- net +5V: track 0.00 -> 13.9 mm
- net Net-(R5-Pad2): track 0.00 -> 3.14 mm
- net Net-(R5-Pad1): track 0.00 -> 3.06 mm
- net GND: vias 0 -> 5
- added copper zone on B.Cu, net GND
- added copper zone on F.Cu, net GND
Other:
- board outline added: 21 x 21.7 mm
